Commit message: parallel training

File: assets/urdf/RobotDog7kg/RobotDog.urdf (robot description, URDF)
Before this commit: robot RobotDog, 9 links, 8 joints
Joints:
- removed joint Revolute_1
- removed joint Revolute_2
- removed joint Revolute_3
- removed joint Revolute_4
- removed joint Revolute_5
- removed joint Revolute_6
- removed joint Revolute_7
- removed joint Revolute_8
- added joint joint_1_0: type revolute, parent base_link, child leg1_1, origin xyz=0.108728 0.076125 0.03886 rpy=0 0 0, axis 0.0 1.0 0.0, limit lower=-2.0944 upper=2.0944 effort=3.8 velocity=5.4
- added joint joint_1_1: type revolute, parent base_link, child leg2_1, origin xyz=-0.134347 0.076125 0.038955 rpy=0 0 0, axis 0.0 1.0 0.0, limit lower=-2.0944 upper=2.0944 effort=3.8 velocity=5.4
- added joint joint_1_2: type revolute, parent base_link, child leg3_1, origin xyz=0.102253 -0.076125 0.041624 rpy=0 0 0, axis 0.0 1.0 0.0, limit lower=-2.0944 upper=2.0944 effort=3.8 velocity=5.4
- added joint joint_1_3: type revolute, parent base_link, child leg4_1, origin xyz=-0.144982 -0.076125 0.03761 rpy=0 0 0, axis 0.0 1.0 0.0, limit lower=-2.0944 upper=2.0944 effort=3.8 velocity=5.4
- added joint joint_2_0: type revolute, parent leg1_1, child foot1_1, origin xyz=-0.000708 0.024408 -0.109869 rpy=0 0 0, axis 0.0 1.0 0.0, limit lower=-2.0944 upper=2.0944 effort=3.8 velocity=5.4
- added joint joint_2_1: type revolute, parent leg2_1, child foot2_1, origin xyz=-0.008066 0.036633 -0.109964 rpy=0 0 0, axis 0.0 1.0 0.0, limit lower=-2.0944 upper=2.0944 effort=3.8 velocity=5.4
- added joint joint_2_2: type revolute, parent leg3_1, child foot3_1, origin xyz=0.00154 -0.035396 -0.112633 rpy=0 0 0, axis 0.0 1.0 0.0, limit lower=-2.0944 upper=2.0944 effort=3.8 velocity=5.4
- added joint joint_2_3: type revolute, parent leg4_1, child foot4_1, origin xyz=0.00138 -0.025554 -0.108619 rpy=0 0 0, axis 0.0 1.0 0.0, limit lower=-2.0944 upper=2.0944 effort=3.8 velocity=5.4

Commit message: updatea urdf name

File: assets/urdf/RobotDog7kg/RobotDog.urdf (robot description, URDF)
Before this commit: robot RobotDog, 9 links, 8 joints
Links:
- removed link foot1_1
- removed link foot2_1
- removed link foot3_1
- removed link foot4_1
- removed link leg1_1
- removed link leg2_1
- removed link leg3_1
- removed link leg4_1
- added link body_1_1_1, mass 0.17635098126357945; collision mesh filename=meshes/leg1_1.stl scale=0.001 0.001 0.001; visual mesh filename=meshes/leg1_1.stl scale=0.001 0.001 0.001
- added link body_1_2_1, mass 0.21988900237553521; collision mesh filename=meshes/leg2_1.stl scale=0.001 0.001 0.001; visual mesh filename=meshes/leg2_1.stl scale=0.001 0.001 0.001
- added link body_1_3_1, mass 0.2124436301601684; collision mesh filename=meshes/leg3_1.stl scale=0.001 0.001 0.001; visual mesh filename=meshes/leg3_1.stl scale=0.001 0.001 0.001
- added link body_1_4_1, mass 0.16803507345033536; collision mesh filename=meshes/leg4_1.stl scale=0.001 0.001 0.001; visual mesh filename=meshes/leg4_1.stl scale=0.001 0.001 0.001
- added link body_2_1_1, mass 0.4197478789995662; collision mesh filename=meshes/foot1_1.stl scale=0.001 0.001 0.001; visual mesh filename=meshes/foot1_1.stl scale=0.001 0.001 0.001
- added link body_2_2_1, mass 0.4725136412635692; collision mesh filename=meshes/foot2_1.stl scale=0.001 0.001 0.001; visual mesh filename=meshes/foot2_1.stl scale=0.001 0.001 0.001
- added link body_2_3_1, mass 0.39949807856162617; collision mesh filename=meshes/foot3_1.stl scale=0.001 0.001 0.001; visual mesh filename=meshes/foot3_1.stl scale=0.001 0.001 0.001
- added link body_2_4_1, mass 0.47989575308955273; collision mesh filename=meshes/foot4_1.stl scale=0.001 0.001 0.001; visual mesh filename=meshes/foot4_1.stl scale=0.001 0.001 0.001
Joints:
- joint joint_1_0: child leg1_1 -> body_1_1_1
- joint joint_1_1: child leg2_1 -> body_1_2_1
- joint joint_1_2: child leg3_1 -> body_1_3_1
- joint joint_1_3: child leg4_1 -> body_1_4_1
- joint joint_2_0: child foot1_1 -> body_2_1_1; parent leg1_1 -> body_1_1_1
- joint joint_2_1: child foot2_1 -> body_2_2_1; parent leg2_1 -> body_1_2_1
- joint joint_2_2: child foot3_1 -> body_2_3_1; parent leg3_1 -> body_1_3_1
- joint joint_2_3: child foot4_1 -> body_2_4_1; parent leg4_1 -> body_1_4_1
