Commit message: add humanoid USD asset for isaac sim

File: assets/urdf/v6biped_urdf_v4_aug29/v6biped_urdf_v4_squarefoot_aug29.urdf (robot description, URDF)
Before this commit: robot v6biped_urdf_v4_squarefoot, 19 links, 18 joints
Links:
- removed link 01_L_hip_z_1
- removed link 02_L_hip_y_1
- removed link 03_L_hip_x_COLLISION_1
- removed link 04_L_knee_rocker_1
- removed link 05_L_knee_link_1
- removed link 06_L_ankle_rocker_1
- removed link 07_L_shank_link_main_1
- removed link 08_L_shank_ankle_link_1
- removed link 09_L_foot_square_COLLISION_1
- removed link 10_R_hip_z_1
- removed link 11_R_hip_y_1
- removed link 12_R_hip_x_COLLISION_1
- removed link 13_R_knee_rocker_1
- removed link 14_R_knee_link_1
- removed link 15_R_ankle_rocker_1
- removed link 16_R_shank_link_main_1
- removed link 17_R_shank_ankle_link_1
- removed link 18_R_foot_square_COLLISION_1
- added link link_01_L_hip_z_1, mass 2.908965938735465; visual mesh filename=meshes/link_01_L_hip_z_1.stl scale=0.001 0.001 0.001
- added link link_02_L_hip_y_1, mass 2.0377990564836805; visual mesh filename=meshes/link_02_L_hip_y_1.stl scale=0.001 0.001 0.001
- added link link_03_L_hip_x_COLLISION_1, mass 3.5805439636700287; collision box size=0.12 0.08 0.27; visual mesh filename=meshes/link_03_L_hip_x_COLLISION_1.stl scale=0.001 0.001 0.001
- added link link_04_L_knee_rocker_1, mass 0.15488700659123303; visual mesh filename=meshes/link_04_L_knee_rocker_1.stl scale=0.001 0.001 0.001
- added link link_05_L_knee_link_1, mass 0.21980714584506778; visual mesh filename=meshes/link_05_L_knee_link_1.stl scale=0.001 0.001 0.001
- added link link_06_L_ankle_rocker_1, mass 0.1199950147888805; visual mesh filename=meshes/link_06_L_ankle_rocker_1.stl scale=0.001 0.001 0.001
- added link link_07_L_shank_link_main_1, mass 0.45787218753949377; visual mesh filename=meshes/link_07_L_shank_link_main_1.stl scale=0.001 0.001 0.001
- added link link_08_L_shank_ankle_link_1, mass 0.2800894766748255; visual mesh filename=meshes/link_08_L_shank_ankle_link_1.stl scale=0.001 0.001 0.001
- added link link_09_L_foot_square_COLLISION_1, mass 0.25; collision mesh filename=meshes/link_09_L_foot_square_COLLISION_1.stl scale=0.001 0.001 0.001; visual mesh filename=meshes/link_09_L_foot_square_COLLISION_1.stl scale=0.001 0.001 0.001
- added link link_10_R_hip_z_1, mass 2.9089659387354665; visual mesh filename=meshes/link_10_R_hip_z_1.stl scale=0.001 0.001 0.001
- added link link_11_R_hip_y_1, mass 2.0377990564836805; visual mesh filename=meshes/link_11_R_hip_y_1.stl scale=0.001 0.001 0.001
- added link link_12_R_hip_x_COLLISION_1, mass 3.5805439636700305; collision box size=0.12 0.08 0.27; visual mesh filename=meshes/link_12_R_hip_x_COLLISION_1.stl scale=0.001 0.001 0.001
- added link link_13_R_knee_rocker_1, mass 0.15488700659123308; visual mesh filename=meshes/link_13_R_knee_rocker_1.stl scale=0.001 0.001 0.001
- added link link_14_R_knee_link_1, mass 0.21980714584506778; visual mesh filename=meshes/link_14_R_knee_link_1.stl scale=0.001 0.001 0.001
- added link link_15_R_ankle_rocker_1, mass 0.11999501478888035; visual mesh filename=meshes/link_15_R_ankle_rocker_1.stl scale=0.001 0.001 0.001
- added link link_16_R_shank_link_main_1, mass 0.45787218753949305; visual mesh filename=meshes/link_16_R_shank_link_main_1.stl scale=0.001 0.001 0.001
- added link link_17_R_shank_ankle_link_1, mass 0.2800894766748255; visual mesh filename=meshes/link_17_R_shank_ankle_link_1.stl scale=0.001 0.001 0.001
- added link link_18_R_foot_square_COLLISION_1, mass 0.25; collision mesh filename=meshes/link_18_R_foot_square_COLLISION_1.stl scale=0.001 0.001 0.001; visual mesh filename=meshes/link_18_R_foot_square_COLLISION_1.stl scale=0.001 0.001 0.001
Joints:
- removed joint 01_L_hip_z
- removed joint 02_L_hip_y
- removed joint 03_L_hip_x
- removed joint 04_L_knee_rocker_RIGID
- removed joint 05_L_knee_link_RIGID
- removed joint 06_L_ankle_rocker_RIGID
- removed joint 07_L_shank_link_main
- removed joint 08_L_shank_ankle_link_RIGID
- removed joint 09_L_foot
- removed joint 10_R_hip_z
- removed joint 11_R_hip_y
- removed joint 12_R_hip_x
- removed joint 13_R_knee_rocker_RIGID
- removed joint 14_R_knee_link_PASSIVE
- removed joint 15_R_ankle_rocker_RIGID
- removed joint 16_R_shank_link_main
- removed joint 17_R_shank_ankle_link_RIGID
- removed joint 18_R_foot
- added joint joint_01_L_hip_z: type revolute, parent base_link, child link_01_L_hip_z_1, origin xyz=0.0 0.09 0.0003 rpy=0 0 0, axis 0.0 0.0 -1.0, limit lower=-1.570796 upper=1.570796 effort=81 velocity=13.333
- added joint joint_02_L_hip_y: type revolute, parent link_01_L_hip_z_1, child link_02_L_hip_y_1, origin xyz=0.0 0.078 -0.0873 rpy=0 0 0, axis 0.0 -1.0 0.0, limit lower=-1.570796 upper=1.570796 effort=90 velocity=12
- added joint joint_03_L_hip_x: type revolute, parent link_02_L_hip_y_1, child link_03_L_hip_x_COLLISION_1, origin xyz=0.0272 -0.077 0.0 rpy=0 0 0, axis 1.0 0.0 0.0, limit lower=-0.628319 upper=0.628319 effort=81 velocity=13.333
- added joint joint_04_L_knee_rocker_RIGID: type fixed, parent link_03_L_hip_x_COLLISION_1, child link_04_L_knee_rocker_1, origin xyz=-0.0302 0.004774 -0.141 rpy=0 0 0
- added joint joint_05_L_knee_link_RIGID: type fixed, parent link_04_L_knee_rocker_1, child link_05_L_knee_link_1, origin xyz=-0.047693 -0.0047 -0.076324 rpy=0 0 0
- added joint joint_06_L_ankle_rocker_RIGID: type fixed, parent link_03_L_hip_x_COLLISION_1, child link_06_L_ankle_rocker_1, origin xyz=-0.0302 -0.008226 -0.281 rpy=0 0 0
- added joint joint_07_L_shank_link_main: type revolute, parent link_03_L_hip_x_COLLISION_1, child link_07_L_shank_link_main_1, origin xyz=-0.0302 0.006574 -0.281 rpy=0 0 0, axis 0.0 1.0 0.0, limit lower=-0.087266 upper=1.745329 effort=81 velocity=13.333
- added joint joint_08_L_shank_ankle_link_RIGID: type fixed, parent link_07_L_shank_link_main_1, child link_08_L_shank_ankle_link_1, origin xyz=0.041681 -0.0065 -0.113024 rpy=0 0 0
- added joint joint_09_L_foot: type revolute, parent link_07_L_shank_link_main_1, child link_09_L_foot_square_COLLISION_1, origin xyz=0.0 -0.0065 -0.235 rpy=0 0 0, axis 0.0 1.0 0.0, limit lower=-0.872665 upper=0.872665 effort=45 velocity=10.667
- added joint joint_10_R_hip_z: type revolute, parent base_link, child link_10_R_hip_z_1, origin xyz=0.0 -0.09 0.0003 rpy=0 0 0, axis 0.0 0.0 -1.0, limit lower=-1.570796 upper=1.570796 effort=81 velocity=13.333
- added joint joint_11_R_hip_y: type revolute, parent link_10_R_hip_z_1, child link_11_R_hip_y_1, origin xyz=0.0 -0.078 -0.0873 rpy=0 0 0, axis 0.0 1.0 0.0, limit lower=-1.570796 upper=1.570796 effort=90 velocity=12
- added joint joint_12_R_hip_x: type revolute, parent link_11_R_hip_y_1, child link_12_R_hip_x_COLLISION_1, origin xyz=0.0272 0.077 0.0 rpy=0 0 0, axis 1.0 0.0 0.0, limit lower=-0.628319 upper=0.628319 effort=81 velocity=13.333
- added joint joint_13_R_knee_rocker_RIGID: type fixed, parent link_12_R_hip_x_COLLISION_1, child link_13_R_knee_rocker_1, origin xyz=-0.0302 -0.004774 -0.141 rpy=0 0 0
- added joint joint_14_R_knee_link_PASSIVE: type fixed, parent link_13_R_knee_rocker_1, child link_14_R_knee_link_1, origin xyz=-0.047693 0.0047 -0.076324 rpy=0 0 0
- added joint joint_15_R_ankle_rocker_RIGID: type fixed, parent link_12_R_hip_x_COLLISION_1, child link_15_R_ankle_rocker_1, origin xyz=-0.0302 0.008226 -0.281 rpy=0 0 0
- added joint joint_16_R_shank_link_main: type revolute, parent link_12_R_hip_x_COLLISION_1, child link_16_R_shank_link_main_1, origin xyz=-0.0302 -0.006574 -0.281 rpy=0 0 0, axis 0.0 -1.0 0.0, limit lower=-1.745329 upper=0.087266 effort=81 velocity=13.333
- added joint joint_17_R_shank_ankle_link_RIGID: type fixed, parent link_16_R_shank_link_main_1, child link_17_R_shank_ankle_link_1, origin xyz=0.041681 0.0065 -0.113024 rpy=0 0 0
- added joint joint_18_R_foot: type revolute, parent link_16_R_shank_link_main_1, child link_18_R_foot_square_COLLISION_1, origin xyz=0.0 0.0065 -0.235 rpy=0 0 0, axis 0.0 -1.0 0.0, limit lower=-0.872665 upper=0.872665 effort=45 velocity=10.667
